File: USB_key_PCB/USB_key_PCB.kicad_pcb (KiCad board)
At the start: 4 copper layers, 12.1 x 14.1 mm, 24 parts, among them U1 STM32F412CEUx, Y1 25MHz

Commit message: Layout start
Parts:
- added C11: 1u, Capacitor_SMD:C_0402_1005Metric, F.Cu at (106.9, 64.9)
- added C12: 1u, Capacitor_SMD:C_0402_1005Metric, F.Cu at (104.7, 64.9)
- added J1: USB, Marijn_KiCad:PCB_USB, F.Cu at (105.8, 57.0)
- added U2: ~, Marijn_KiCad:X2-DFN1010-4, F.Cu at (105.8, 65.0)
- C1, C10, C2, C3, C4, C5, C6, C7, C8, C9: footprint Capacitor_SMD:C_0603_1608Metric -> Capacitor_SMD:C_0402_1005Metric
- L1: footprint Inductor_SMD:L_0805_2012Metric -> Inductor_SMD:L_0402_1005Metric
- R1, R2, R3: footprint Resistor_SMD:R_0603_1608Metric -> Resistor_SMD:R_0402_1005Metric
- moved TP5 42.1 mm to (100.7, 74.7)
- moved TP6 41.8 mm to (100.7, 76.7)
- moved Y1 41.2 mm to (105.8, 76.0)
- moved C6 35.9 mm to (102.7, 76.6)
- moved TP7 35.6 mm to (111.0, 76.7)
- moved TP1 34.9 mm to (100.7, 65.0)
- moved R1 34.8 mm to (101.1, 68.8), turned to -90 degrees
- moved TP8 34.3 mm to (111.0, 74.7)
- moved L1 33.5 mm to (110.5, 72.8), turned to -90 degrees
- moved R3 33.1 mm to (101.1, 70.8), turned to 90 degrees
- moved TP2 33.1 mm to (102.7, 65.0)
- moved R2 32.5 mm to (108.5, 76.2), turned to 90 degrees
- moved TP4 29.8 mm to (109.0, 65.0)
- moved C9 29.2 mm to (103.2, 75.2), turned to 90 degrees
- moved C7 28.6 mm to (109.0, 74.7), turned to 180 degrees
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Connections:
- C2 pad 1: +3.3V -> +3V3
- C3 pad 1: +3.3V -> +3V3
- C4 pad 1: +3.3V -> +3V3
- C5 pad 1: +3.3V -> +3V3
- C6 pad 1: +3.3V -> +3V3
- L1 pad 1: +3.3V -> +3V3
- TP5 pad 1: unconnected-(TP5-Pad1) -> +3V3
- TP6 pad 1: unconnected-(TP6-Pad1) -> /SWCLK
- TP7 pad 1: unconnected-(TP7-Pad1) -> /SWDIO
- TP8 pad 1: unconnected-(TP8-Pad1) -> GND
- U1 pad 1: +3.3V -> +3V3
- U1 pad 24: +3.3V -> +3V3
- U1 pad 36: +3.3V -> +3V3
- U1 pad 48: +3.3V -> +3V3
Routing:
- net GND: track 0.00 -> 61.2 mm, vias 0 -> 12
- net +3V3: track 0.00 -> 20.5 mm, vias 0 -> 5
- net /NRST: track 0.00 -> 20.3 mm, vias 0 -> 3
- net +5V: track 0.00 -> 13.5 mm
- net /BOOT0: track 0.00 -> 8.17 mm
- net /HSE_OUT: track 0.00 -> 6.36 mm, vias 0 -> 2
- net /HSE_IN: track 0.00 -> 5.91 mm, vias 0 -> 2
- net +3.3VA: track 0.00 -> 5.08 mm
- net Net-(C10-Pad1): track 0.00 -> 2.79 mm
- net Net-(U1-VCAP_1): track 0.00 -> 1.71 mm
- added copper zone on In1.Cu, net +5V
- added copper zone on B.Cu, net GND
- added copper zone on F.Cu, net GND
- added copper zone on In2.Cu, net GND
Other:
- board size 12.1 x 14.1 mm -> 12.1 x 28.1 mm
