File: USB_key_PCB/USB_key_PCB.kicad_sch (KiCad schematic)
At the start: 24 parts, among them U1 STM32F412CEUx, Y1 25MHz

Commit message: Layout start
Parts:
- added C11, C12: 1u, Capacitor_SMD:C_0402_1005Metric, symbol Device:C_Small
- added J1: USB, Marijn_KiCad:PCB_USB, symbol Connector:USB_A
- added U2: ~, Marijn_KiCad:X2-DFN1010-4, symbol Marijn:AP7343D-33W5
- C1, C10, C2, C3, C4, C5, C6, C7, C8, C9: footprint Capacitor_SMD:C_0603_1608Metric -> Capacitor_SMD:C_0402_1005Metric
- L1: footprint Inductor_SMD:L_0805_2012Metric -> Inductor_SMD:L_0402_1005Metric
- R1, R2, R3: footprint Resistor_SMD:R_0603_1608Metric -> Resistor_SMD:R_0402_1005Metric
Connections:
- net +3.3V is gone; now on net +3V3: C2.1, C3.1, C4.1, C5.1, C6.1, L1.1, U1.1 (VBAT), U1.24 (VDD), U1.36 (VDD), U1.48 (VDD)
- net +3V3: now also TP5.1, C12.1, U2.5 (VOUT)
- net GND: now also TP8.1, C11.2, C12.2, J1.4 (GND), U2.2 (GND)
- net SWCLK: now reaches TP6.1
- net SWDIO: now reaches TP7.1
- new net +5V: C11.1, J1.1 (VBUS), U2.1 (VIN), U2.3 (EN)
- new net USB_DN: J1.2 (D-)
- new net USB_DP: J1.3 (D+)
- no-connect marks 0 -> 1
